File: sd-card-adapter/sd-adapter.kicad_pcb (KiCad board)
At the start: 2 copper layers, 14.2 x 31 mm, 9 parts, among them J101 Conn_01x01_Male, J102 Conn_01x01_Male, J103 Conn_01x01_Male, J104 Conn_01x01_Male, J105 Conn_01x01_Male, J106 Conn_01x01_Male, J107 Conn_01x01_Male, J108 Conn_01x01_Male

Commit message: Removal of host port and preparation for manufacturing
Other:
- board text added: "PCB thickness 1mm"
Changed lines of the file:
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@@
   (general
     (thickness 1.6)
-    (drawings 22)
+    (drawings 23)
     (tracks 213)
     (modules 9)
@@
     (39 "F.Mask" user)
     (40 "Dwgs.User" user hide)
-    (41 "Cmts.User" user hide)
+    (41 "Cmts.User" user)
     (42 "Eco1.User" user)
     (43 "Eco2.User" user)
@@
       (dielectric_constraints no)
     )
-    (last_trace_width 0.17)
+    (last_trace_width 0.25)
     (user_trace_width 0.17)
     (user_trace_width 0.25)
@@
       (net 8 "/DAT1S") (pinfunction "Pin_1"))
   )
+  (gr_text "PCB thickness 1mm" (at 164.88 101.84) (layer "Cmts.User")
+    (effects (font (size 1 1) (thickness 0.15)))
+  )
   (gr_text "Armbian\nuSD\nadapter" (at 150.8 111.8) (layer "F.SilkS")
